File: 01-2x30w_audio_amp/01-2x30w_audio_amp.kicad_pcb (KiCad board)
At the start: 4 copper layers, 49.8 x 49.8 mm, 103 parts, among them J1 CUI 3.5mm, J2 CUI 3.5mm, J3 Conn_02x07_Odd_Even, J4 CUI 3.5mm, U1 TL071HIDBVR, U2 LM317L_SOT-89, U3 TL331BIDBVR, U4 TPA3118D2, U5 TL071HIDBVR

Commit message: Minor tweaks
Parts:
- added R34: inf, Resistor_SMD:R_0603_1608Metric, B.Cu at (179.3, 96.7)
- moved R26 3.00 mm to (182.3, 96.7)
- moved R25 2.34 mm to (183.1, 98.9), turned to 90 degrees
Routing:
- net +24V: track 33.0 -> 30.4 mm
- net Net-(U4-MODSEL): track 6.02 -> 3.96 mm
- net Net-(C14-Pad1): track 3.02 -> 4.64 mm
Other:
- board text added: "Pegboard 01 v1.0 2x30W Audio Amp"
- board text removed: "Pegboard 01 2x30W Audio Amp"
