File: 01-2x30w_audio_amp/01-2x30w_audio_amp.kicad_sch (KiCad schematic)
At the start: 103 parts, among them J1 CUI 3.5mm, J2 CUI 3.5mm, J3 Conn_02x07_Odd_Even, J4 CUI 3.5mm, U1 TL071HIDBVR, U2 LM317L_SOT-89, U3 TL331BIDBVR, U4 TPA3118D2, U5 TL071HIDBVR

Commit message: Minor tweaks
Parts:
- added R34: inf, Resistor_SMD:R_0603_1608Metric, symbol Device:R_Small
Connections:
- net GND: now also R34.2
- net at C14.1, C9.2, R16.2: now also R34.1
Other:
- moved on the sheet: R16
